File: Electrical/Buisness Card.kicad_sch (KiCad schematic)
At the start: 75 parts, among them IC1 74HC595, IC2 74HC595, Q1 BC547, Q2 BC547, Q3 BC547, Q4 BC547, Q5 BC547, Q6 BC547, Q7 BC547, Q8 BC547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

Commit message: directory changes
Connections:
- net at Q7.2 (B): no longer IC2.6 (QG)
- net at D25.A, D26.A, D27.A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: no longer IC1.3 (QD)
- net at D1.A, D2.A, D3.A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: no longer IC1.15 (QA)
- net at D10.A, D11.A, D12.A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: no longer IC1.1 (QB)
- net at D36.A, D40.A, D44.A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: no longer IC1.7 (QH)
- net at D35.A, D39.A, D43.A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: no longer IC1.6 (QG)
- net at D17.A, D18.A, D19.A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: no longer IC1.2 (QC)
- net at D33.A, D37.A, D41.A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: no longer IC1.4 (QE)
- net at D34.A, D38.A, D42.A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: no longer IC1.5 (QF)
- net at Q5.2 (B): no longer IC2.4 (QE)
- net at Q8.2 (B): no longer IC2.7 (QH)
- net at Q1.2 (B): no longer IC2.15 (QA)
- net at Q6.2 (B): no longer IC2.5 (QF)
- net at IC2.1 (QB): no longer Q2.2 (B)
- net at IC2.2 (QC): no longer Q3.2 (B)
- net at IC2.3 (QD): no longer Q4.2 (B)
